Commit message: mm

File: polymetis/polymetis/data/franka_panda/panda_arm.urdf (robot description, URDF)
Before this commit: robot panda, 9 links, 8 joints
Links:
- added link panda_hand, mass 0.73; collision mesh filename=meshes/collision/hand.stl; visual mesh filename=meshes/visual/hand.dae
- added link panda_leftfinger, mass 0.015; collision mesh filename=meshes/collision/finger.stl; visual mesh filename=meshes/visual/finger.dae
- added link panda_rightfinger, mass 0.015; collision mesh filename=meshes/collision/finger.stl; visual mesh filename=meshes/visual/finger.dae
- added link panda_tool
Joints:
- added joint panda_finger_joint1: type fixed, parent panda_hand, child panda_leftfinger, origin xyz=0 0 0.0584 rpy=0 0 0, axis 0 1 0, limit lower=-0.001 upper=0.04 effort=20 velocity=0.3
- added joint panda_finger_joint2: type fixed, parent panda_hand, child panda_rightfinger, origin xyz=0 0 0.0584 rpy=0 0 0, axis 0 -1 0, limit lower=-0.001 upper=0.04 effort=20 velocity=0.3
- added joint panda_hand_joint: type fixed, parent panda_link8, child panda_hand, origin xyz=0 0 0 rpy=0 0 -0.785398163397
- added joint panda_hand_tool_joint: type fixed, parent panda_hand, child panda_tool, origin xyz=0 0 0.1034 rpy=0 0 0
